File: TP4056_4cell_charger.kicad_pcb (KiCad board)
At the start: 2 copper layers, 110 x 135 mm, 57 parts, among them J1 Screw_Terminal_01x02, U1 TP4056-42-ESOP8, U2 TP4056-42-ESOP8, U3 TP4056-42-ESOP8, U4 TP4056-42-ESOP8

Commit message: finished v1 final version
Parts:
- added C12: 220n, Capacitor_SMD:C_0603_1608Metric, F.Cu at (166.8, 59.2)
- added C3: 220n, Capacitor_SMD:C_0603_1608Metric, F.Cu at (92.2, 59.2)
- added C6: 220n, Capacitor_SMD:C_0603_1608Metric, F.Cu at (117.2, 59.2)
- added C9: 220n, Capacitor_SMD:C_0603_1608Metric, F.Cu at (142.2, 59.2)
- added J2: CellHolder_4x18650_Parallel, JK_footprints:4xCellHolder_18650, F.Cu at (138.1, 119.1)
- moved TH4 19.6 mm to (174.6, 98.8)
- moved TH1 18.6 mm to (101.7, 98.8)
- moved TH3 8.80 mm to (155.2, 119.1)
- moved TH2 5.87 mm to (121.0, 119.1)
- moved TP1 3.02 mm to (110.6, 169.1)
- moved TP2 3.02 mm to (105.6, 169.1)
- moved TP3 3.02 mm to (130.6, 169.1)
- moved TP4 3.02 mm to (125.6, 169.1)
- moved TP5 3.02 mm to (150.6, 169.1)
- moved TP6 3.02 mm to (145.6, 169.1)
- moved TP7 3.02 mm to (170.6, 169.1)
- moved TP8 3.02 mm to (165.6, 169.1)
- moved C2 2.31 mm to (100.7, 68.6)
- moved C5 2.31 mm to (125.7, 68.6)
- moved C11 2.31 mm to (175.7, 68.6)
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- renumbered C7 to C10, C8 to C11, C3 to C4, C4 to C5, C5 to C7, C6 to C8, H3 to H2, H2 to H3, R4 to R1, R9 to R10, R12 to R11, R15 to R12, R11 to R13, R13 to R14, R14 to R15, R17 to R16, R20 to R17, R16 to R18, R18 to R19, R3 to R2, R19 to R20, R2 to R3, R1 to R4, R7 to R6, R10 to R7, R6 to R8, R8 to R9
Connections:
- net Net-(BT1-+) renamed /Charger1/Bat_Out
- net Net-(BT2-+) renamed /Charger2/Bat_Out
- net Net-(BT3-+) renamed /Charger3/Bat_Out
- net Net-(BT4-+) renamed /Charger4/Bat_Out
Routing:
- net GND: track 35.5 -> 220.6 mm, vias 18 -> 93
- net /Charger4/Bat_Out: track 0.00 -> 114.8 mm
- net /Charger3/Bat_Out: track 0.00 -> 110.7 mm, vias 0 -> 2
- net /Charger1/Bat_Out: track 0.00 -> 110.7 mm, vias 0 -> 2
- net /Charger2/Bat_Out: track 0.00 -> 108.7 mm, vias 0 -> 2
- net Net-(U3-TEMP): track 16.8 -> 76.3 mm, vias 2 -> 4
- net Net-(U2-TEMP): track 16.8 -> 70.7 mm
- net Net-(U4-TEMP): track 17.2 -> 59.0 mm, vias 2 -> 4
- net Net-(U1-TEMP): track 16.8 -> 52.7 mm
Other:
- board text added: "STNB"
- board text removed: "DCHRG"
