File: TP4056_4cell_charger.kicad_sch (KiCad schematic)
At the start: 5 parts, among them J1 Screw_Terminal_01x02

Commit message: finished v1 final version
Parts:
- added J2: CellHolder_4x18650_Parallel, JK_footprints:4xCellHolder_18650, symbol JK_symbols:CellHolder_18650_4x_Parallel
- renumbered H3 to H2, H2 to H3
Connections:
- net GND: now also J2.5 (B1-), J2.6 (B2-), J2.7 (B3-), J2.8 (B4-)
- new net Charger1/Bat_Out: J2.1 (B1+)
- new net Charger2/Bat_Out: J2.2 (B2+)
- new net Charger3/Bat_Out: J2.3 (B3+)
- new net Charger4/Bat_Out: J2.4 (B4+)
Other:
- sheet Charger1 ports: added Bat_Out; removed none
- sheet Charger2 ports: added Bat_Out; removed none
- sheet Charger3 ports: added Bat_Out; removed none
- sheet Charger4 ports: added Bat_Out; removed none
- moved on the sheet: J1
