File: untitled.kicad_sch (KiCad schematic)
At the start: 14 parts, among them U1 TP4056-42-ESOP8

Commit message: finished v1 final version
Parts:
- added C3: 220n, Capacitor_SMD:C_0603_1608Metric, symbol Device:C
- BT1: now not fitted; now left out of the parts list
- renumbered R4 to R1, R3 to R2, R2 to R3, R1 to R4
Connections:
- net GND: now also C3.2
- net Bat_Out: now reaches BT1.1 (+), C2.1, TP1.1, U1.5 (BAT)
- net at R2.2, R5.1, TH1.1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: now also C3.1
Other:
- moved on the sheet: C2, R2, R4, R5, TH1
