File: Li-Ion_18650_Holder_Series_Board/Li_Ion_18650_Holder_Series_Board/Li_Ion_18650_Holder_Series_Board.kicad_pcb (KiCad board)
At the start: 2 copper layers, 7 parts, among them J2 Conn_01x01_Pin, J3 Conn_01x01_Pin

Commit message: working on layout
Parts:
- moved F4 17.4 mm to (153.2, 135.8), turned to -90 degrees
- moved J3 2.92 mm to (157.2, 141.8)
Routing:
- net B+: track 0.00 -> 11.9 mm
- net B4+: track 0.00 -> 6.27 mm
Other:
- board outline added: 100 x 100 mm
Changed lines of the file:
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@@
 	(footprint "Fuse:Fuse_0603_1608Metric"
 		(layer "F.Cu")
-		(at 164.2125 149.25)
+		(at 153.25 135.75 -90)
 		(descr "Fuse SMD 0603 (1608 Metric), square (rectangular) end terminal, IPC-7351 nominal, (Body size source: http://www.tortai-tech.com/upload/download/2011102023233369053.pdf), generated with kicad-footprint-generator")
 		(tags "fuse")
 		(property "Reference" "F4"
-			(at 0 -1.43 0)
+			(at 0 -1.43 90)
 			(layer "F.SilkS")
 			(effects
@@
 		)
 		(property "Value" "Fuse"
-			(at 0 1.43 0)
+			(at 0 1.43 90)
 			(layer "F.Fab")
 			(effects
@@
 		)
 		(property "Datasheet" "~"
-			(at 0 0 0)
+			(at 0 0 90)
 			(layer "F.Fab")
 			(hide yes)
@@
 		)
 		(property "Description" "Fuse"
-			(at 0 0 0)
+			(at 0 0 90)
 			(layer "F.Fab")
 			(hide yes)
@@
 		)
 		(property "LCSC" "C41380234"
-			(at 0 0 0)
+			(at 0 0 270)
 			(unlocked yes)
 			(layer "F.Fab")
@@
 		(attr smd)
 		(fp_line
+			(start -0.162779 0.51)
+			(end 0.162779 0.51)
+			(stroke
+				(width 0.12)
+				(type solid)
+			)
+			(layer "F.SilkS")
+		)
+		(fp_line
 			(start -0.162779 -0.51)
 			(end 0.162779 -0.51)
@@
 		)
 		(fp_line
-			(start -0.162779 0.51)
-			(end 0.162779 0.51)
-			(stroke
-				(width 0.12)
-				(type solid)
-			)
-			(layer "F.SilkS")
+			(start -1.48 0.73)
+			(end -1.48 -0.73)
+			(stroke
+				(width 0.05)
+				(type solid)
+			)
+			(layer "F.CrtYd")
+		)
+		(fp_line
+			(start 1.48 0.73)
+			(end -1.48 0.73)
+			(stroke
+				(width 0.05)
+				(type solid)
+			)
+			(layer "F.CrtYd")
 		)
 		(fp_line
@@
 		)
 		(fp_line
-			(start -1.48 0.73)
-			(end -1.48 -0.73)
-			(stroke
-				(width 0.05)
-				(type solid)
-			)
-			(layer "F.CrtYd")
-		)
-		(fp_line
 			(start 1.48 -0.73)
 			(end 1.48 0.73)
@@
 		)
 		(fp_line
-			(start 1.48 0.73)
-			(end -1.48 0.73)
-			(stroke
-				(width 0.05)
-				(type solid)
-			)
-			(layer "F.CrtYd")
+			(start -0.8 0.4)
+			(end -0.8 -0.4)
+			(stroke
+				(width 0.1)
+				(type solid)
+			)
+			(layer "F.Fab")
+		)
+		(fp_line
+			(start 0.8 0.4)
+			(end -0.8 0.4)
+			(stroke
+				(width 0.1)
+				(type solid)
+			)
+			(layer "F.Fab")
 		)
 		(fp_line
@@
 		)
 		(fp_line
-			(start -0.8 0.4)
-			(end -0.8 -0.4)
-			(stroke
-				(width 0.1)
-				(type solid)
-			)
-			(layer "F.Fab")
-		)
-		(fp_line
 			(start 0.8 -0.4)
 			(end 0.8 0.4)
@@
 			(layer "F.Fab")
 		)
-		(fp_line
-			(start 0.8 0.4)
-			(end -0.8 0.4)
-			(stroke
-				(width 0.1)
-				(type solid)
-			)
-			(layer "F.Fab")
-		)
 		(fp_text user "${REFERENCE}"
-			(at 0 0 0)
+			(at 0 0 90)
 			(layer "F.Fab")
 			(effects
@@
 		)
 		(pad "1" smd roundrect
-			(at -0.7875 0)
+			(at -0.7875 0 270)
 			(size 0.875 0.95)
 			(layers "F.Cu" "F.Mask" "F.Paste")
@@
 		)
 		(pad "2" smd roundrect
-			(at 0.7875 0)
+			(at 0.7875 0 270)
 			(size 0.875 0.95)
 			(layers "F.Cu" "F.Mask" "F.Paste")
@@
 	(footprint "JK_footprints:Faston_C27636945"
 		(layer "F.Cu")
-		(at 159.75 143.25)
+		(at 157.25 141.75)
 		(property "Reference" "J3"
 			(at 0 -0.5 0)
@@
 		(net 1)
 	)
+	(gr_rect
+		(start 79.5 46)
+		(end 179.5 146)
+		(stroke
+			(width 0.2)
+			(type solid)
+		)
+		(fill no)
+		(layer "Edge.Cuts")
+	)
 	(segment
 		(start 99.5 136.318019)
@@
 		(net 7)
 	)
+	(segment
+		(start 159.5 135)
+		(end 153.2875 135)
+		(width 1)
+		(layer "F.Cu")
+		(net 8)
+	)
+	(segment
+		(start 153.2875 135)
+		(end 153.25 134.9625)
+		(width 1)
+		(layer "F.Cu")
+		(net 8)
+	)
+	(segment
+		(start 153.25 136.5375)
+		(end 153.25 137.75)
+		(width 1)
+		(layer "F.Cu")
+		(net 9)
+	)
+	(segment
+		(start 153.25 137.75)
+		(end 157.25 141.75)
+		(width 1)
+		(layer "F.Cu")
+		(net 9)
+	)
+	(segment
+		(start 157.25 141.75)
+		(end 162.25 141.75)
+		(width 1)
+		(layer "F.Cu")
+		(net 9)
+	)
 	(embedded_fonts no)
